File: hardware/electric-imp-breakout.brd (EAGLE design)
At the start: 32.1 x 50.8 mm, 22 parts, among them Q1 DMG2307L-7, U1 ELECTRIC_IMP, U2 TPS62172, U3 ATSHA204-TSU, X1 USBSMD

Commit message: changed micro fid to regular
Parts:
- removed JP8, JP9: FIDUCIALUFIDUCIAL, SparkFun:MICRO-FIDUCIAL
- added FID1, FID2: FIDUCIAL1X2, SparkFun-Aesthetics:FIDUCIAL-1X2
